File: Sicherungskarte.kicad_pcb (KiCad board)
At the start: 2 copper layers, 52 x 56 mm, 12 parts, among them J1 MKDS_3-3_5.08, J2 MKDS_3-3_5.08, J3 MKDS_3-3_5.08, J4 MKDS_3-3_5.08

Commit message: final version
Routing:
- net Net-(J2-Pin_1): track 0.00 -> 36.2 mm
- net Net-(J4-Pin_3): track 0.00 -> 35.7 mm
- net Net-(J3-Pin_1): track 0.00 -> 35.7 mm
- net Net-(J2-Pin_3): track 0.00 -> 35.7 mm
- net Net-(J1-Pin_3): track 0.00 -> 35.7 mm
- net Net-(J1-Pin_1): track 0.00 -> 35.7 mm
- net Net-(J4-Pin_1): track 0.00 -> 35.7 mm
- net Net-(J3-Pin_3): track 0.00 -> 35.7 mm
- net Net-(J2-Pin_2): track 0.00 -> 33.3 mm
- net Net-(J1-Pin_2): track 0.00 -> 33.3 mm
- net Net-(J4-Pin_2): track 0.00 -> 33.3 mm
- net Net-(J3-Pin_2): track 0.00 -> 33.3 mm
Other:
- board text added: "10A max / Fuse"
